Commit message: feat(controller): 添加深度强化学习控制器支持及传感器配置
refactor(description): 重构机器人描述文件，移除冗余相机配置

build: 更新CMakeLists和package.xml，添加OpenCV等依赖

docs(config): 新增并更新配置文件，优化参数说明

test(worlds): 添加带传感器的仿真世界文件，支持深度相机测试

fix(launch): 修复启动文件问题，优化节点启动顺序和参数传递

style: 统一代码格式，增加必要注释和日志输出

File: descriptions/peak_lab/depth_go2_description/xacro/gazebo.xacro (robot description, xacro)
@@ -144,4 +144,12 @@
       <state_interface name="RL_foot_force"/>
     </sensor>
+    <sensor name="odometer">
+      <state_interface name="position.x"/>
+      <state_interface name="position.y"/>
+      <state_interface name="position.z"/>
+      <state_interface name="velocity.x"/>
+      <state_interface name="velocity.y"/>
+      <state_interface name="velocity.z"/>
+    </sensor>
   </ros2_control>
   <gazebo>
@@ -232,35 +240,6 @@
     <xacro:include filename="$(find gz_quadruped_playground)/models/D435/model.xacro"/>
     <xacro:d435 camID="1" name="d435">
-      <origin rpy="0 0.1 0" xyz="0.28 0 0.093"/>
+      <origin rpy="0 0.2 0" xyz="0.30 0 0.10"/>
     </xacro:d435>
-    <gazebo reference="front_camera">
-      <sensor name="front_camera" type="camera">
-        <camera>
-          <horizontal_fov>2.094</horizontal_fov>
-          <image>
-            <width>1280</width>
-            <height>720</height>
-          </image>
-          <clip>
-            <near>0.1</near>
-            <far>15</far>
-          </clip>
-          <noise>
-            <type>gaussian</type>
-            <!-- Noise is sampled independently per pixel on each frame.
-                That pixel's noise value is added to each of its color
-                channels, which at that point lie in the range [0,1]. -->
-            <mean>0.0</mean>
-            <stddev>0.007</stddev>
-          </noise>
-          <optical_frame_id>front_camera</optical_frame_id>
-          <camera_info_topic>camera/camera_info</camera_info_topic>
-        </camera>
-        <always_on>true</always_on>
-        <update_rate>15</update_rate>
-        <visualize>true</visualize>
-        <topic>camera/image</topic>
-      </sensor>
-    </gazebo>
     <gazebo reference="lidar">
       <sensor name='L1_lidar' type='gpu_lidar'>

File: descriptions/peak_lab/depth_go2_description/xacro/robot.xacro (robot description, xacro)
@@ -7,5 +7,4 @@
   <xacro:include filename="$(find depth_go2_description)/xacro/materials.xacro"/>
   <xacro:include filename="$(find depth_go2_description)/xacro/leg.xacro"/>
-  <xacro:include filename="$(find realsense2_description)/urdf/_d435i.urdf.xacro"/>
   <xacro:if value="$(arg GAZEBO)">
     <xacro:if value="$(arg CLASSIC)">
@@ -39,7 +38,4 @@
     </visual>
   </link>
-  <xacro:sensor_d435i parent="base" name="depth_camera" use_nominal_extrinsics="false">
-        <origin xyz="0.27 0 0.08" rpy="0 0 0"/>
-  </xacro:sensor_d435i>
   <joint name="floating_base" type="fixed">
     <origin rpy="0 0 0" xyz="0 0 0"/>
@@ -113,11 +109,4 @@
     </collision>
   </link>
-  <joint name="camera_joint_front" type="fixed">
-    <parent link="trunk"/>
-    <child link="front_camera"/>
-    <origin rpy="0 0 0" xyz="0.32715 0 0.04297"/>
-  </joint>
-  <link name="front_camera">
-  </link>
   <joint name="lidar_joint" type="fixed">
     <origin

Commit message: feat(controller): 添加新的深度强化学习控制器及相关配置
- 新增our_depth_rl_quadruped_controller控制器，支持基于深度相机的四足机器人控制。
- 实现了状态机管理和深度图像处理功能，优化了控制器的参数配置。
- 更新了CMakeLists.txt和package.xml以包含新的依赖项。
- 添加了多个配置文件和启动文件，支持在Gazebo和Mujoco中进行仿真。
- 引入了低通滤波器和观测缓存机制，提升了控制精度和稳定性。
- 更新了README文档，提供了编译和使用说明。

File: descriptions/peak_lab/depth_go2_description/xacro/gazebo.xacro (robot description, xacro)
@@ -240,5 +240,5 @@
     <xacro:include filename="$(find gz_quadruped_playground)/models/D435/model.xacro"/>
     <xacro:d435 camID="1" name="d435">
-      <origin rpy="0 0.2 0" xyz="0.30 0 0.10"/>
+      <origin rpy="0 $(arg CAMERA_PITCH) 0" xyz="0.24 0 0.12"/>
     </xacro:d435>
     <gazebo reference="lidar">

File: descriptions/peak_lab/depth_go2_description/xacro/robot.xacro (robot description, xacro)
@@ -4,4 +4,5 @@
   <xacro:arg name="GAZEBO" default="false"/>
   <xacro:arg name="CLASSIC" default="false"/>
+  <xacro:arg name="CAMERA_PITCH" default="0.0"/>
   <xacro:include filename="$(find depth_go2_description)/xacro/const.xacro"/>
   <xacro:include filename="$(find depth_go2_description)/xacro/materials.xacro"/>

Commit message: feat(controller): 更新深度强化学习控制器及相关配置
- 在StateRL中添加了新的参数以支持深度图像处理和动作输出的低通滤波。
- 引入了新的深度图像预处理逻辑，增强了对无效深度帧的处理能力。
- 更新了模型参数配置，增加了前进命令速度和DOF重排选项。
- 新增了MuJoCo视觉测试启动文件，简化了仿真环境的启动流程。
- 调整了Gazebo和深度相机的配置，优化了相机位置和传感器设置。
- 更新了相关文档以反映新的配置和功能。

File: descriptions/peak_lab/depth_go2_description/xacro/gazebo.xacro (robot description, xacro)
@@ -236,9 +236,9 @@
   <xacro:foot_force_sensor name="FR" suffix="foot_fixed"/>
   <xacro:foot_force_sensor name="RR" suffix="foot_fixed"/>
-  <xacro:arg name="EXTERNAL_SENSORS" default="false"/>
+  <xacro:arg name="EXTERNAL_SENSORS" default="true"/>
   <xacro:if value="$(arg EXTERNAL_SENSORS)">
     <xacro:include filename="$(find gz_quadruped_playground)/models/D435/model.xacro"/>
     <xacro:d435 camID="1" name="d435">
-      <origin rpy="0 $(arg CAMERA_PITCH) 0" xyz="0.24 0 0.12"/>
+      <origin rpy="0 0 0" xyz="0.32 0 0.09"/>
     </xacro:d435>
     <gazebo reference="lidar">

File: descriptions/peak_lab/depth_go2_description/xacro/robot.xacro (robot description, xacro)
@@ -4,5 +4,5 @@
   <xacro:arg name="GAZEBO" default="false"/>
   <xacro:arg name="CLASSIC" default="false"/>
-  <xacro:arg name="CAMERA_PITCH" default="0.0"/>
+  <xacro:arg name="CAMERA_PITCH" default="-0.25"/>
   <xacro:include filename="$(find depth_go2_description)/xacro/const.xacro"/>
   <xacro:include filename="$(find depth_go2_description)/xacro/materials.xacro"/>

Commit message: feat(controller): 增强深度强化学习控制器功能与配置
- 在StateRL中添加了关节和足端的重排参数，支持ROS顺序到策略顺序的映射。
- 引入onboard模型加载功能，允许使用onboard策略进行推理。
- 更新深度图像预处理逻辑，优化无效深度帧的处理。
- 调整Gazebo和深度相机的配置，优化相机位置和传感器设置。
- 更新配置文件，替换旧模型文件名并添加新的模型文件。
- 修复启动文件中的图像桥接问题，确保深度图像正常传输。

File: descriptions/peak_lab/depth_go2_description/xacro/gazebo.xacro (robot description, xacro)
@@ -1,4 +1,6 @@
 <?xml version="1.0"?>
 <robot xmlns:xacro="http://www.ros.org/wiki/xacro">
+  <!-- 供相机安装角度使用；由上层 robot.xacro 传入时会覆盖默认值 -->
+  <xacro:arg name="CAMERA_PITCH" default="0.0"/>
   <xacro:include filename="$(find gz_quadruped_hardware)/xacro/foot_force_sensor.xacro"/>
   <ros2_control name="GazeboSystem" type="system">
@@ -240,5 +242,5 @@
     <xacro:include filename="$(find gz_quadruped_playground)/models/D435/model.xacro"/>
     <xacro:d435 camID="1" name="d435">
-      <origin rpy="0 0 0" xyz="0.32 0 0.09"/>
+      <origin rpy="0 0.4 0" xyz="0.32 0 0.09"/>
     </xacro:d435>
     <gazebo reference="lidar">

File: libraries/gz_quadruped_playground/models/D435/model.xacro (robot description, xacro)
@@ -58,10 +58,10 @@
           <clip>
             <near>0.01</near>
-            <far>300</far>
+            <far>10.0</far>
           </clip>
           <depth_camera>
             <clip>
-              <near>0.1</near>
-              <far>10</far>
+              <near>0.01</near>
+              <far>10.0</far>
             </clip>
           </depth_camera>

Commit message: fix

File: descriptions/peak_lab/depth_go2_description/xacro/gazebo.xacro (robot description, xacro)
@@ -242,5 +242,6 @@
     <xacro:include filename="$(find gz_quadruped_playground)/models/D435/model.xacro"/>
     <xacro:d435 camID="1" name="d435">
-      <origin rpy="0 0.4 0" xyz="0.32 0 0.09"/>
+      <!-- <origin rpy="0 0.1 0" xyz="0.32 0 0.09"/> -->
+      <origin rpy="0 0.2 0" xyz="0.24 0 0.12"/>
     </xacro:d435>
     <gazebo reference="lidar">

Commit message: add some config

File: descriptions/peak_lab/depth_go2_description/xacro/gazebo.xacro (robot description, xacro)
@@ -243,5 +243,5 @@
     <xacro:d435 camID="1" name="d435">
       <!-- <origin rpy="0 0.1 0" xyz="0.32 0 0.09"/> -->
-      <origin rpy="0 0.2 0" xyz="0.24 0 0.12"/>
+      <origin rpy="0 0.1 0" xyz="0.24 0 0.12"/>
     </xacro:d435>
     <gazebo reference="lidar">

Commit message: Successfully depolyment

File: descriptions/peak_lab/depth_go2_description/xacro/gazebo.xacro (robot description, xacro)
@@ -242,6 +242,7 @@
     <xacro:include filename="$(find gz_quadruped_playground)/models/D435/model.xacro"/>
     <xacro:d435 camID="1" name="d435">
-      <!-- <origin rpy="0 0.1 0" xyz="0.32 0 0.09"/> -->
-      <origin rpy="0 0.1 0" xyz="0.24 0 0.12"/>
+      <!-- 与该 checkpoint 的 config.json 对齐：position=[0.24,0,0.12], angle=[0,1]°
+           原值 pitch=0.2rad(11.5°) 远超训练范围 [0°,1°]，改为 0° -->
+      <origin rpy="0 0.0 0" xyz="0.24 0 0.12"/>
     </xacro:d435>
     <gazebo reference="lidar">

File: descriptions/peak_lab/depth_go2_description/xacro/ros2_control.xacro (robot description, xacro)
@@ -4,6 +4,7 @@
 		<hardware>
 			<plugin>hardware_unitree_sdk2/HardwareUnitree</plugin>
+			<!-- DDS：与实机一致。domain 通常 0 或 1；network_interface 为本机连机器人的网卡（ifconfig 查看），如 eth0、eth6 -->
 			<param name="domain">0</param>
-			<param name="network_interface">eth2</param>
+			<param name="network_interface">eth0</param>
 			<param name="show_foot_force">false</param>
 		</hardware>
@@ -140,9 +141,10 @@
 			<state_interface name="linear_acceleration.z"/>
 		</sensor>
+		<!-- 与 gazebo.xacro 一致：FL_foot_force 等，保证仿真/实机共用同一套 robot_control.yaml -->
 		<sensor name="foot_force">
-			<state_interface name="FR"/>
-			<state_interface name="FL"/>
-			<state_interface name="RR"/>
-			<state_interface name="RL"/>
+			<state_interface name="FR_foot_force"/>
+			<state_interface name="FL_foot_force"/>
+			<state_interface name="RR_foot_force"/>
+			<state_interface name="RL_foot_force"/>
 		</sensor>
 		<sensor name="odometer">

File: libraries/gz_quadruped_playground/models/D435/model.xacro (robot description, xacro)
@@ -33,5 +33,6 @@
       <sensor name="realsense_d435" type="rgbd_camera">
         <camera name="d435">
-          <horizontal_fov>1.0472</horizontal_fov>
+          <!-- 与训练端 legged_robot_config.py depth.horizontal_fov=87° 对齐；原值 1.0472(60°) 视野过窄 -->
+          <horizontal_fov>1.518</horizontal_fov>
           <lens>
             <intrinsics>
